Commit message: added moveit

File: src/kuka_agilus_description/urdf/kr6_r900_2.urdf (robot description, URDF)
Before this commit: robot kr6_r900_2, 11 links, 10 joints
Links:
- added link suction_cup, mass 7.34E-1; collision mesh filename=package://kuka_agilus_description/meshes/kr6_r900_2/collisi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 scale=0.002 0.002 0.002; visual mesh filename=package://kuka_agilus_description/meshes/kr6_r900_2/visual/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 scale=0.002 0.002 0.002
Joints:
- added joint tool0-suction: type fixed, parent tool0, child suction_cup, origin xyz=0.0 0.0 -0.0285 rpy=3.141592653589793 1.2246467991473532E-16 3.141592653589793

File: src/kuka_agilus_description/urdf/kr6_r900_2_macro.xacro (robot description, xacro)
@@ -137,4 +137,26 @@
       </visual>
     </link>
+    <link name = "suction_cup">
+      <collision>
+        <geometry>
+          <mesh filename="package://kuka_agilus_description/meshes/kr6_r900_2/collision/suction_head.stl" scale = "0.002 0.002 0.002"/>
+        </geometry>
+        <origin rpy="1.2246467991473532e-16 3.141592653589793 0.0" xyz="0.0 -1.941931457395624e-17 -0.025"/>
+      </collision>
+      <inertial>
+        <inertia ixx="1.83698267603013E-4" ixy="0.0" ixz="0.0" iyy="1.8213621766783165E-4" iyz="0.0" izz="2.9589000000000004E-4"/>
+        <mass value="7.34E-1"/>
+        <origin rpy="0.0 -0.0 1.223427188696551" xyz="0.0 0.0 -0.011764604904632152"/>
+      </inertial>
+      <visual>
+        <geometry>
+          <mesh filename="package://kuka_agilus_description/meshes/kr6_r900_2/visual/suction_head.stl" scale = "0.002 0.002 0.002"/>
+        </geometry>
+        <origin rpy="1.2246467991473532e-16 3.141592653589793 0.0" xyz="0.0 -1.941931457395624e-17 -0.025"/>
+        <material name="bodyTextured_material">
+                <color rgba="0.0 0.0 0.506 1.0" />
+      </material>
+      </visual>
+    </link>
     <link name="${prefix}tool0"/>
     <joint name="${prefix}base_link-base" type="fixed">
@@ -194,4 +216,9 @@
       <parent link="${prefix}link_6"/>
     </joint>
+    <joint name="tool0-suction" type="fixed">
+      <child link="suction_cup"/>
+      <origin rpy="3.141592653589793 1.2246467991473532E-16 3.141592653589793" xyz="0.0 0.0 -0.0285"/>
+      <parent link="tool0"/>
+    </joint>
   </xacro:macro>
 </robot>
