Commit message: added camera

File: src/kuka_agilus_description/urdf/kr6_r900_2.urdf.xacro (robot description, xacro)
@@ -3,4 +3,5 @@
   <!-- Import macro files  -->
   <xacro:include filename="$(find kuka_agilus_description)/urdf/kr6_r900_2_macro.xacro"/>
+  <xacro:include filename="$(find kuka_agilus_description)/urdf/kuka_camera.xacro"/>
   <xacro:include filename="$(find kuka_agilus_description)/urdf/kr_agilus_ros2_control_macro.xacro"/>
   <!-- Read additional arguments  -->
@@ -24,4 +25,8 @@
     <ext_axes_ros2_control_joints/>
   </xacro:kuka_agilus_ros2_control>
+  <xacro:camera_v0 parent="base_link">
+	    <origin xyz="0.2 0.6 0.7" rpy="0 ${PI/2} 0"/>
+  </xacro:camera_v0>
+  <xacro:camera_gazebo_v0/>
   <!-- world link -->
   <link name="world"/>
