Commit message: ur5

File: src/robot_description/urdf/ur5.urdf.xacro (robot description, xacro)
@@ -184,250 +184,396 @@
     <limit lower="-6.28319" upper="6.28319" effort="28.0" velocity="3.2"/>
   </joint>
-  <joint name="robotiq_85_base_joint" type="fixed">
+  <joint name="robotiq_140_base_joint" type="fixed">
       <parent link="wrist_3_link"/>
-      <child link="robotiq_85_base_link"/>
-      <origin xyz="0 0.0823 0" rpy="1.570796325 0 1.570796325"/>
+      <child link="robotiq_140_base_link"/>
+      <origin xyz="0 0.0823 0" rpy="1.570796325 0 3.141592653"/>
       <limit lower="0" upper="0" effort="0" velocity="0"/>
     </joint>
-    <link name="robotiq_85_base_link">
-      <visual>
-        <geometry>
-          <mesh filename="package://robot_description/meshes/ur5/visual/robotiq_85_base_link.dae"/>
-        </geometry>
-      </visual>
-      <collision>
-        <geometry>
-          <mesh filename="package://robot_description/meshes/ur5/collision/robotiq_85_base_link.stl"/>
-        </geometry>
-      </collision>
-      <inertial>
-        <mass value="0.636951" />
-        <origin xyz="0.0 0.0 0.0" />
-        <inertia ixx = "0.000380" ixy = "0.000000" ixz = "0.000000"
-             iyx = "0.000000" iyy = "0.001110" iyz = "0.000000"
-             izx = "0.000000" izy = "0.000000" izz = "0.001171" />
-      </inertial>
-    </link>
-    <joint name="robotiq_85_left_knuckle_joint" type="revolute">
-      <parent link="robotiq_85_base_link"/>
-      <child link="robotiq_85_left_knuckle_link"/>
-      <axis xyz="0 0 1"/>
-      <origin rpy="${pi} 0.0 0.0" xyz="0.05490451627 0.03060114443 0.0"/>
-      <limit lower="0.0" upper="0.80285" velocity="0.5" effort="1000"/>
-    </joint>
-    <joint name="robotiq_85_right_knuckle_joint" type="continuous">
-      <parent link="robotiq_85_base_link"/>
-      <child link="robotiq_85_right_knuckle_link"/>
-      <axis xyz="0 0 1"/>
-      <origin rpy="0.0 0.0 0.0" xyz="0.05490451627 -0.03060114443 0.0"/>
-      <limit lower="-3.14" upper="3.14" velocity="100.0" effort="1000"/>
-      <mimic joint="robotiq_85_left_knuckle_joint"/>
-    </joint>
-     <link name="robotiq_85_left_knuckle_link">
-      <visual>
-        <geometry>
-          <mesh filename="package://robot_description/meshes/ur5/visual/robotiq_85_knuckle_link.dae"/>
-        </geometry>
-      </visual>
-      <collision>
-        <geometry>
-          <mesh filename="package://robot_description/meshes/ur5/collision/robotiq_85_knuckle_link.stl"/>
-        </geometry>
-      </collision>
-      <inertial>
-        <mass value="0.018491" />
-        <origin xyz="0.0 0.0 0.0" />
-        <inertia ixx = "0.000009" ixy = "-0.000001" ixz = "0.000000"
-             iyx = "-0.000001" iyy = "0.000010" iyz = "0.000000"
-             izx = "0.000000" izy = "0.000000" izz = "0.000010" />
-      </inertial>
-    </link>
-    <link name="robotiq_85_right_knuckle_link">
-      <visual>
-        <geometry>
-          <mesh filename="package://robot_description/meshes/ur5/visual/robotiq_85_knuckle_link.dae"/>
-        </geometry>
-      </visual>
-      <collision>
-        <geometry>
-          <mesh filename="package://robot_description/meshes/ur5/collision/robotiq_85_knuckle_link.stl"/>
-        </geometry>
-      </collision>
-      <inertial>
-        <mass value="0.018491" />
-        <origin xyz="0.0 0.0 0.0" />
-        <inertia ixx = "0.000009" ixy = "-0.000001" ixz = "0.000000"
-             iyx = "-0.000001" iyy = "0.000010" iyz = "0.000000"
-             izx = "0.000000" izy = "0.000000" izz = "0.000010" />
-      </inertial>
-    </link>
-    <joint name="robotiq_85_left_finger_joint" type="fixed">
-      <parent link="robotiq_85_left_knuckle_link"/>
-      <child link="robotiq_85_left_finger_link"/>
-      <origin xyz="-0.00408552455 -0.03148604435 0.0" rpy="0 0 0" />
-    </joint>
-    <joint name="robotiq_85_right_finger_joint" type="fixed">
-      <parent link="robotiq_85_right_knuckle_link"/>
-      <child link="robotiq_85_right_finger_link"/>
-      <origin xyz="-0.00408552455 -0.03148604435 0.0" rpy="0 0 0" />
-    </joint>
-    <link name="robotiq_85_left_finger_link">
-      <visual>
-        <geometry>
-          <mesh filename="package://robot_description/meshes/ur5/visual/robotiq_85_finger_link.dae"/>
-        </geometry>
-      </visual>
-      <collision>
-        <geometry>
-          <mesh filename="package://robot_description/meshes/ur5/collision/robotiq_85_finger_link.stl"/>
-        </geometry>
-      </collision>
-      <inertial>
-        <mass value="0.027309" />
-        <origin xyz="0.0 0.0 0.0" />
-        <inertia ixx = "0.000003" ixy = "-0.000002" ixz = "0.000000"
-             iyx = "-0.000002" iyy = "0.000021" iyz = "0.000000"
-             izx = "0.000000" izy = "0.000000" izz = "0.000020" />
-      </inertial>
-    </link>
-    <link name="robotiq_85_right_finger_link">
-      <visual>
-        <geometry>
-          <mesh filename="package://robot_description/meshes/ur5/visual/robotiq_85_finger_link.dae"/>
-        </geometry>
-      </visual>
-      <collision>
-        <geometry>
-          <mesh filename="package://robot_description/meshes/ur5/collision/robotiq_85_finger_link.stl"/>
-        </geometry>
-      </collision>
-      <inertial>
-        <mass value="0.027309" />
-        <origin xyz="0.0 0.0 0.0" />
-        <inertia ixx = "0.000003" ixy = "-0.000002" ixz = "0.000000"
-             iyx = "-0.000002" iyy = "0.000021" iyz = "0.000000"
-             izx = "0.000000" izy = "0.000000" izz = "0.000020" />
-      </inertial>
-    </link>
-    <joint name="robotiq_85_left_inner_knuckle_joint" type="continuous">
-      <parent link="robotiq_85_base_link"/>
-      <child link="robotiq_85_left_inner_knuckle_link"/>
-      <axis xyz="0 0 1"/>
-      <origin xyz="0.06142 0.0127 0" rpy="${pi} 0.0 0.0" />
-      <limit lower="-3.14" upper="3.14" velocity="100.0" effort="0.1"/>
-      <mimic joint="robotiq_85_left_knuckle_joint" offset="0"/>
-    </joint>
-    <joint name="robotiq_85_right_inner_knuckle_joint" type="continuous">
-      <parent link="robotiq_85_base_link"/>
-      <child link="robotiq_85_right_inner_knuckle_link"/>
-      <axis xyz="0 0 1"/>
-      <origin xyz="0.06142 -0.0127 0" rpy="0 0 0"/>
-      <limit lower="-3.14" upper="3.14" velocity="100.0" effort="0.1"/>
-      <mimic joint="robotiq_85_left_knuckle_joint" offset="0"/>
-    </joint>
-    <link name="robotiq_85_left_inner_knuckle_link">
-      <visual>
-        <geometry>
-          <mesh filename="package://robot_description/meshes/ur5/visual/robotiq_85_inner_knuckle_link.dae"/>
-        </geometry>
-      </visual>
-      <collision>
-        <geometry>
-          <mesh filename="package://robot_description/meshes/ur5/collision/robotiq_85_inner_knuckle_link.stl"/>
-        </geometry>
-      </collision>
-      <inertial>
-        <mass value="0.029951" />
-        <origin xyz="0.0 0.0 0.0" />
-        <inertia ixx = "0.000039" ixy = "0.000000" ixz = "0.000000"
-             iyx = "0.000000" iyy = "0.000005" iyz = "0.000000"
-             izx = "0.000000" izy = "0.000000" izz = "0.000035" />
-      </inertial>
-    </link>
-    <link name="robotiq_85_right_inner_knuckle_link">
-      <visual>
-        <geometry>
-          <mesh filename="package://robot_description/meshes/ur5/visual/robotiq_85_inner_knuckle_link.dae"/>
-        </geometry>
-      </visual>
-      <collision>
-        <geometry>
-          <mesh filename="package://robot_description/meshes/ur5/collision/robotiq_85_inner_knuckle_link.stl"/>
-        </geometry>
-      </collision>
-      <inertial>
-        <mass value="0.029951" />
-        <origin xyz="0.0 0.0 0.0" />
-        <inertia ixx = "0.000039" ixy = "0.000000" ixz = "0.000000"
-             iyx = "0.000000" iyy = "0.000005" iyz = "0.000000"
-             izx = "0.000000" izy = "0.000000" izz = "0.000035" />
-      </inertial>
-    </link>
-    <joint name="robotiq_85_left_finger_tip_joint" type="continuous">
-      <parent link="robotiq_85_left_inner_knuckle_link"/>
-      <child link="robotiq_85_left_finger_tip_link"/>
-      <axis xyz="0 0 1"/>
-      <origin xyz="0.04303959807 -0.03759940821 0.0" rpy="0.0 0.0 0.0"/>
-      <limit lower="-3.14" upper="3.14" velocity="100.0" effort="0.1"/>
-      <mimic joint="robotiq_85_left_knuckle_joint" multiplier="-1"/>
-    </joint>
-    <joint name="robotiq_85_right_finger_tip_joint" type="continuous">
-      <parent link="robotiq_85_right_inner_knuckle_link"/>
-      <child link="robotiq_85_right_finger_tip_link"/>
-      <axis xyz="0 0 1"/>
-      <origin rpy="0.0 0.0 0.0" xyz="0.04303959807 -0.03759940821  0.0"/>
-      <limit lower="-3.14" upper="3.14" velocity="100.0" effort="0.1"/>
-      <mimic joint="robotiq_85_left_knuckle_joint" multiplier="-1"/>
-    </joint>
-     <link name="robotiq_85_left_finger_tip_link">
-      <visual>
-        <geometry>
-          <mesh filename="package://robot_description/meshes/ur5/visual/robotiq_85_finger_tip_link.dae"/>
-        </geometry>
-      </visual>
-      <collision>
-        <geometry>
-          <mesh filename="package://robot_description/meshes/ur5/collision/robotiq_85_finger_tip_link.stl"/>
-        </geometry>
-      </collision>
-      <inertial>
-        <mass value="0.019555" />
-        <origin xyz="0.0 0.0 0.0" />
-        <inertia ixx = "0.000002" ixy = "0.000000" ixz = "0.000000"
-             iyx = "0.000000" iyy = "0.000005" iyz = "0.000000"
-             izx = "0.000000" izy = "0.000000" izz = "0.000006" />
-      </inertial>
-    </link>
-    <link name="robotiq_85_right_finger_tip_link">
-      <visual>
-        <geometry>
-          <mesh filename="package://robot_description/meshes/ur5/visual/robotiq_85_finger_tip_link.dae"/>
-        </geometry>
-      </visual>
-      <collision>
-        <geometry>
-          <mesh filename="package://robot_description/meshes/ur5/collision/robotiq_85_finger_tip_link.stl"/>
-        </geometry>
-      </collision>
-      <inertial>
-        <mass value="0.019555" />
-        <origin xyz="0.0 0.0 0.0" />
-        <inertia ixx = "0.000002" ixy = "0.000000" ixz = "0.000000"
-             iyx = "0.000000" iyy = "0.000005" iyz = "0.000000"
-             izx = "0.000000" izy = "0.000000" izz = "0.000006" />
-      </inertial>
-    </link>
-    <xacro:include filename="$(find robot_description)/urdf/gazebo_camera.xacro"/>
+  <link name="robotiq_140_base_link">
+    <inertial>
+      <origin rpy="0 0 0" xyz="8.625E-08 -4.6583E-06 0.03145"/>
+      <mass value="0.22652"/>
+      <inertia ixx="0.00020005" ixy="-4.2442E-10" ixz="-2.9069E-10" iyy="0.00017832" iyz="-3.4402E-08" izz="0.00013478"/>
+    </inertial>
+    <visual>
+      <origin rpy="0 0 0" xyz="0 0 0"/>
+      <geometry>
+        <mesh filename="package://robot_description/meshes/ur5/visual/robotiq_arg2f_base_link.stl"/>
+      </geometry>
+      <material name="">
+        <color rgba="0.1 0.1 0.1 1"/>
+      </material>
+    </visual>
+    <collision>
+      <origin rpy="0 0 0" xyz="0 0 0"/>
+      <geometry>
+        <mesh filename="package://robot_description/meshes/ur5/collision/robotiq_arg2f_base_link.stl"/>
+      </geometry>
+    </collision>
+  </link>
+  <link name="left_outer_knuckle">
+    <inertial>
+      <origin rpy="0 0 0" xyz="-0.000200000000003065 0.0199435877845359 0.0292245259211331"/>
+      <mass value="0.00853198276973456"/>
+      <inertia ixx="2.89328108496468E-06" ixy="-1.57935047237397E-19" ixz="-1.93980378593255E-19" iyy="1.86719750325683E-06" iyz="-1.21858577871576E-06" izz="1.21905238907251E-06"/>
+    </inertial>
+    <visual>
+      <origin rpy="0 0 0" xyz="0 0 0"/>
+      <geometry>
+        <mesh filename="package://robot_description/meshes/ur5/visual/robotiq_arg2f_140_outer_knuckle.stl"/>
+      </geometry>
+      <material name="">
+        <color rgba="0.792156862745098 0.819607843137255 0.933333333333333 1"/>
+      </material>
+    </visual>
+    <collision>
+      <origin rpy="0 0 0" xyz="0 0 0"/>
+      <geometry>
+        <mesh filename="package://robot_description/meshes/ur5/collision/robotiq_arg2f_140_outer_knuckle.stl"/>
+      </geometry>
+    </collision>
+  </link>
+  <link name="left_outer_finger">
+    <inertial>
+      <origin rpy="0 0 0" xyz="0.00030115855001899 0.0373907951953854 -0.0208027427000385"/>
+      <mass value="0.022614240507152"/>
+      <inertia ixx="1.52518312458174E-05" ixy="9.76583423954399E-10" ixz="-5.43838577022588E-10" iyy="6.17694243867776E-06" iyz="6.78636130740228E-06" izz="1.16494917907219E-05"/>
+    </inertial>
+    <visual>
+      <origin rpy="0 0 0" xyz="0 0 0"/>
+      <geometry>
+        <mesh filename="package://robot_description/meshes/ur5/visual/robotiq_arg2f_140_outer_finger.stl"/>
+      </geometry>
+      <material name="">
+        <color rgba="0.1 0.1 0.1 1"/>
+      </material>
+    </visual>
+    <collision>
+      <origin rpy="0 0 0" xyz="0 0 0"/>
+      <geometry>
+        <mesh filename="package://robot_description/meshes/ur5/collision/robotiq_arg2f_140_outer_finger.stl"/>
+      </geometry>
+    </collision>
+  </link>
+  <link name="left_inner_finger">
+    <inertial>
+      <origin rpy="0 0 0" xyz="0.000299999999999317 0.0160078233491243 -0.0136945669206257"/>
+      <mass value="0.0104003125914103"/>
+      <inertia ixx="2.71909453810972E-06" ixy="1.35402465472579E-21" ixz="-7.1817349065269E-22" iyy="7.69100314106116E-07" iyz="6.74715432769696E-07" izz="2.30315190420171E-06"/>
+    </inertial>
+    <visual>
+      <origin rpy="0 0 0" xyz="0 0 0"/>
+      <geometry>
+        <mesh filename="package://robot_description/meshes/ur5/visual/robotiq_arg2f_140_inner_finger.stl"/>
+      </geometry>
+      <material name="">
+        <color rgba="0.1 0.1 0.1 1"/>
+      </material>
+    </visual>
+    <collision>
+      <origin rpy="0 0 0" xyz="0 0 0"/>
+      <geometry>
+        <mesh filename="package://robot_description/meshes/ur5/collision/robotiq_arg2f_140_inner_finger.stl"/>
+      </geometry>
+    </collision>
+  </link>
+  <link name="left_inner_finger_pad">
+    <visual>
+      <origin rpy="0 0 0" xyz="0 0 0"/>
+      <geometry>
+        <box size="0.027 0.065 0.0075"/>
+      </geometry>
+      <material name="">
+        <color rgba="0.9 0.9 0.9 1"/>
+      </material>
+    </visual>
+    <collision>
+      <origin rpy="0 0 0" xyz="0 0 0"/>
+      <geometry>
+        <box size="0.03 0.07 0.0075"/>
+      </geometry>
+      <material name="">
+        <color rgba="0.9 0.0 0.0 1"/>
+      </material>
+    </collision>
+  </link>
+  <link name="left_inner_knuckle">
+    <inertial>
+      <origin rpy="0 0 0" xyz="0.000123011831763771 0.0507850843201817 0.00103968640075166"/>
+      <mass value="0.0271177346495152"/>
+      <inertia ixx="2.61910379223783E-05" ixy="-2.43616858946494E-07" ixz="-6.37789906117123E-09" iyy="2.8270243746167E-06" iyz="-5.37200748039765E-07" izz="2.83695868220296E-05"/>
+    </inertial>
+    <visual>
+      <origin rpy="0 0 0" xyz="0 0 0"/>
+      <geometry>
+        <mesh filename="package://robot_description/meshes/ur5/visual/robotiq_arg2f_140_inner_knuckle.stl"/>
+      </geometry>
+      <material name="">
+        <color rgba="0.1 0.1 0.1 1"/>
+      </material>
+    </visual>
+    <collision>
+      <origin rpy="0 0 0" xyz="0 0 0"/>
+      <geometry>
+        <mesh filename="package://robot_description/meshes/ur5/collision/robotiq_arg2f_140_inner_knuckle.stl"/>
+      </geometry>
+    </collision>
+  </link>
+  <link name="right_outer_knuckle">
+    <inertial>
+      <origin rpy="0 0 0" xyz="-0.000200000000003065 0.0199435877845359 0.0292245259211331"/>
+      <mass value="0.00853198276973456"/>
+      <inertia ixx="2.89328108496468E-06" ixy="-1.57935047237397E-19" ixz="-1.93980378593255E-19" iyy="1.86719750325683E-06" iyz="-1.21858577871576E-06" izz="1.21905238907251E-06"/>
+    </inertial>
+    <visual>
+      <origin rpy="0 0 0" xyz="0 0 0"/>
+      <geometry>
+        <mesh filename="package://robot_description/meshes/ur5/visual/robotiq_arg2f_140_outer_knuckle.stl"/>
+      </geometry>
+      <material name="">
+        <color rgba="0.792156862745098 0.819607843137255 0.933333333333333 1"/>
+      </material>
+    </visual>
+    <collision>
+      <origin rpy="0 0 0" xyz="0 0 0"/>
+      <geometry>
+        <mesh filename="package://robot_description/meshes/ur5/collision/robotiq_arg2f_140_outer_knuckle.stl"/>
+      </geometry>
+    </collision>
+  </link>
+  <link name="right_outer_finger">
+    <inertial>
+      <origin rpy="0 0 0" xyz="0.00030115855001899 0.0373907951953854 -0.0208027427000385"/>
+      <mass value="0.022614240507152"/>
+      <inertia ixx="1.52518312458174E-05" ixy="9.76583423954399E-10" ixz="-5.43838577022588E-10" iyy="6.17694243867776E-06" iyz="6.78636130740228E-06" izz="1.16494917907219E-05"/>
+    </inertial>
+    <visual>
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