Commit message: added contact sensor

File: src/robot_description/urdf/kr_agilus_ros2_control_macro.xacro (robot description, xacro)
@@ -4,6 +4,6 @@
     <!-- gazebo -->
     <xacro:if value="${mode == 'gazebo'}">
-      <xacro:include filename="$(find kuka_agilus_description)/urdf/kuka_gazebo.xacro"/>
-      <xacro:kuka_gazebo controller_config_package="kuka_agilus_controller" controller_config_path="config/ros2_controllers.yaml"/>
+      <xacro:include filename="$(find robot_description)/urdf/kuka_gazebo.xacro"/>
+      <xacro:kuka_gazebo controller_config_package="robot_controller" controller_config_path="config/ros2_controllers.yaml"/>
     </xacro:if>
     <!-- ros2 control -->

File: src/robot_description/urdf/kuka_gazebo.xacro (robot description, xacro)
@@ -11,3 +11,17 @@
     </gazebo>
   </xacro:macro>
+  <gazebo reference="tool0-suction">
+  <preserveFixedJoint>true</preserveFixedJoint>
+</gazebo>
+ <gazebo reference="suction_cup">
+          <sensor name="contact_sensor" type="contact">
+            <contact>
+              <collision>suction_cup_collision</collision>
+              <topic>/contact_sensor</topic>
+            </contact>
+            <always_on>true</always_on>
+            <update_rate>30</update_rate>
+            <visualize>true</visualize>
+        </sensor>
+  </gazebo>
 </robot>

File: src/robot_description/urdf/ur5.urdf (robot description, URDF)
Before this commit: robot ur5_robot, 19 links, 18 joints
Links:
- removed link world
Joints:
- removed joint connect_root_and_world
